File: SEQ ISA/_autosave-SEQ ISA.kicad_sch (KiCad schematic)
At the start: 70 parts, among them IC1 TLX9310_TPL,F, IC2 SN74LVC4245ADW, J1 FTSH-107-01-L-DV-K-A, J2 Conn_01x02_Pin, J3 Conn_01x02_Pin, J4 Conn_01x02_Pin, J5 Conn_01x02_Pin, J6 Conn_01x02_Pin, J7 Jack-DC, J8 Conn_01x04_Pin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

Commit message: PCB First version
Connections:
- net PC14: now also J8.1 (Pin_3); no longer J8.3 (Pin_3)
- net PC15: now also J8.2 (Pin_4); no longer J8.4 (Pin_4)
- net PH0: now also J8.3 (Pin_1); no longer J8.1 (Pin_1)
- net PH1: now also J8.4 (Pin_2); no longer J8.2 (Pin_2)
